Commit message: #1 updated the rrbot urdf to create a scara robot (rrp)

File: rrbot_simulation_files/rrbot_description/gazebo/rrbot.gazebo.xacro (robot description, xacro)
@@ -12,9 +12,9 @@
       </plugin>
     </gazebo>
-    <!-- Link1 -->
+    <!-- Base Link -->
     <gazebo reference="${prefix}base_link">
       <material>Gazebo/Orange</material>
     </gazebo>
-    <!-- Link2 -->
+    <!-- Link1 -->
     <gazebo reference="${prefix}link1">
       <mu1>0.2</mu1>
@@ -22,5 +22,5 @@
       <material>Gazebo/Black</material>
     </gazebo>
-    <!-- Link3 -->
+    <!-- Link2 -->
     <gazebo reference="${prefix}link2">
       <mu1>0.2</mu1>
@@ -28,4 +28,10 @@
       <material>Gazebo/Orange</material>
     </gazebo>
+    <!-- Link3 -->
+    <gazebo reference="${prefix}link3">
+      <mu1>0.2</mu1>
+      <mu2>0.2</mu2>
+      <material>Gazebo/Black</material>
+    </gazebo>
   </xacro:macro>
 </robot>

File: rrbot_simulation_files/rrbot_description/urdf/rrbot_description.urdf.xacro (robot description, xacro)
@@ -5,7 +5,8 @@
   <xacro:property name="mass" value="1" /> <!-- arbitrary value for mass -->
   <xacro:property name="width" value="0.1" /> <!-- Square dimensions (widthxwidth) of beams -->
-  <xacro:property name="height1" value="2" /> <!-- Link 1 -->
-  <xacro:property name="height2" value="1" /> <!-- Link 2 -->
-  <xacro:property name="height3" value="1" /> <!-- Link 3 -->
+  <xacro:property name="base_height" value="1.5" /> <!-- Base Link -->
+  <xacro:property name="height1" value="1" /> <!-- Link 1 -->
+  <xacro:property name="height2" value="0.5" /> <!-- Link 2 -->
+  <xacro:property name="height3" value="0.5" /> <!-- Link 3 -->
   <xacro:property name="camera_link" value="0.05" /> <!-- Size of square 'camera' box -->
   <xacro:property name="axel_offset" value="0.05" /> <!-- Space btw top of beam and the each joint -->
@@ -18,67 +19,104 @@
   <link name="${prefix}base_link">
     <collision>
-      <origin xyz="0 0 ${height1/2}" rpy="0 0 0"/>
+      <origin xyz="0 0 ${base_height/2}" rpy="0 0 0"/>
       <geometry>
-        <box size="${width} ${width} ${height1}"/>
+        <box size="${width} ${width} ${base_height}"/>
       </geometry>
     </collision>
     <visual>
-      <origin xyz="0 0 ${height1/2}" rpy="0 0 0"/>
+      <origin xyz="0 0 ${base_height/2}" rpy="0 0 0"/>
       <geometry>
-        <box size="${width} ${width} ${height1}"/>
+        <box size="${width} ${width} ${base_height}"/>
       </geometry>
       <material name="orange"/>
     </visual>
     <inertial>
-      <origin xyz="0 0 ${height1/2}" rpy="0 0 0"/>
+      <origin xyz="0 0 ${base_height/2}" rpy="0 0 0"/>
       <mass value="${mass}"/>
       <inertia
-        ixx="${mass / 12.0 * (width*width + height1*height1)}" ixy="0.0" ixz="0.0"
-        iyy="${mass / 12.0 * (height1*height1 + width*width)}" iyz="0.0"
+        ixx="${mass / 12.0 * (width*width + base_height*base_height)}" ixy="0.0" ixz="0.0"
+        iyy="${mass / 12.0 * (base_height*base_height + width*width)}" iyz="0.0"
         izz="${mass / 12.0 * (width*width + width*width)}"/>
       </inertial>
     </link>
-    <joint name="${prefix}joint1" type="continuous">
+    <!-- First Revolute Joint-->
+    <joint name="${prefix}joint1" type="revolute">
       <parent link="${prefix}base_link"/>
       <child link="${prefix}link1"/>
-      <origin xyz="0 ${width} ${height1 - axel_offset}" rpy="0 1.5708 0"/>
-      <axis xyz="1 0 0"/>
+      <origin xyz="0 0 ${base_height + axel_offset}" rpy="0 0 0"/>
+      <axis xyz="0 0 1"/>
       <dynamics damping="0.7"/>
+      <limit effort="300" velocity="0.1" lower="-3.14" upper="3.14"/>
     </joint>
-    <!-- Middle Link -->
+    <!-- Link 1 -->
     <link name="${prefix}link1">
       <collision>
-        <origin xyz="0 0 ${height2/2 - axel_offset}" rpy="0 0 0"/>
+        <origin xyz="${height1/2 - axel_offset} 0 0" rpy="0 0 0"/>
         <geometry>
-          <box size="${width} ${width} ${height2}"/>
+          <box size="$${height1} ${width} ${width}"/>
         </geometry>
       </collision>
       <visual>
-        <origin xyz="0 0 ${height2/2 - axel_offset}" rpy="0 0 0"/>
+        <origin xyz="${height1/2 - axel_offset} 0 0" rpy="0 0 0"/>
         <geometry>
-          <box size="${width} ${width} ${height2}"/>
+          <box size="${height1} ${width} ${width}"/>
         </geometry>
         <material name="yellow"/>
       </visual>
       <inertial>
-        <origin xyz="0 0 ${height2/2 - axel_offset}" rpy="0 0 0"/>
+        <origin xyz="${height1/2 - axel_offset} 0 0" rpy="0 0 0"/>
         <mass value="${mass}"/>
         <inertia
-          ixx="${mass / 12.0 * (width*width + height2*height2)}" ixy="0.0" ixz="0.0"
-          iyy="${mass / 12.0 * (height2*height2 + width*width)}" iyz="0.0"
-          izz="${mass / 12.0 * (width*width + width*width)}"/>
+          ixx="${mass / 12.0 * (width*width + width*width)}" ixy="0.0" ixz="0.0"
+          iyy="${mass / 12.0 * (height1*height1 + width*width)}" iyz="0.0"
+          izz="${mass / 12.0 * (width*width + height1*height1)}"/>
         </inertial>
       </link>
-      <joint name="${prefix}joint2" type="continuous">
+      <!-- Second Revolute Joint -->
+      <joint name="${prefix}joint2" type="revolute">
         <parent link="${prefix}link1"/>
         <child link="${prefix}link2"/>
-        <origin xyz="0 ${width} ${height2 - axel_offset*2}" rpy="0 0 0"/>
-        <axis xyz="1 0 0"/>
+        <origin xyz="${height1 - axel_offset*2} 0 ${-width}" rpy="0 0 0"/>
+        <axis xyz="0 0 1"/>
         <dynamics damping="0.7"/>
+        <limit effort="300" velocity="0.1" lower="-3.14" upper="3.14"/>
       </joint>
-      <!-- Top Link -->
+      <!-- Link 2 -->
       <link name="${prefix}link2">
         <collision>
-          <origin xyz="0 0 ${height3/2 - axel_offset}" rpy="0 0 0"/>
+          <origin xyz="${height2/2 - axel_offset} 0 0" rpy="0 0 0"/>
+          <geometry>
+            <box size="${height2} ${width} ${width}"/>
+          </geometry>
+        </collision>
+        <visual>
+          <origin xyz="${height2/2 - axel_offset} 0 0" rpy="0 0 0"/>
+          <geometry>
+            <box size="${height2} ${width} ${width}"/>
+          </geometry>
+          <material name="orange"/>
+        </visual>
+        <inertial>
+          <origin xyz="${height2/2 - axel_offset} 0 0" rpy="0 0 0"/>
+          <mass value="${mass}"/>
+          <inertia
+            ixx="${mass / 12.0 * (width*width + width*width)}" ixy="0.0" ixz="0.0"
+            iyy="${mass / 12.0 * (height2*height2 + width*width)}" iyz="0.0"
+            izz="${mass / 12.0 * (width*width + height2*height2)}"/>
+          </inertial>
+        </link>
+      <!-- Prismatic Joint -->
+      <joint name="${prefix}joint3" type="prismatic">
+        <parent link="${prefix}link2"/>
+        <child link="${prefix}link3"/>
+        <origin xyz="${height2 - axel_offset*2} 0 ${-width}" rpy="0 0 0"/>
+        <axis xyz="0 0 -1"/>
+        <dynamics damping="0.7"/>
+        <limit effort="300" velocity="0.1" lower="0" upper="0.50"/>
+      </joint>
+      <!-- Link 3 -->
+      <link name="${prefix}link3">
+        <collision>
+          <origin xyz="0 0 ${-(height3/2 - axel_offset)}" rpy="0 0 0"/>
           <geometry>
             <box size="${width} ${width} ${height3}"/>
@@ -86,12 +124,12 @@
         </collision>
         <visual>
-          <origin xyz="0 0 ${height3/2 - axel_offset}" rpy="0 0 0"/>
+          <origin xyz="0 0 ${-(height3/2 - axel_offset)}" rpy="0 0 0"/>
           <geometry>
             <box size="${width} ${width} ${height3}"/>
           </geometry>
-          <material name="orange"/>
+          <material name="yellow"/>
         </visual>
         <inertial>
-          <origin xyz="0 0 ${height3/2 - axel_offset}" rpy="0 0 0"/>
+          <origin xyz="0 0 ${-(height3/2 - axel_offset)}" rpy="0 0 0"/>
           <mass value="${mass}"/>
           <inertia
@@ -101,7 +139,8 @@
           </inertial>
         </link>
+        <!-- Tool Joint -->
         <joint name="${prefix}tool_joint" type="fixed">
-          <origin xyz="0 0 1" rpy="0 0 0" />
-          <parent link="${prefix}link2"/>
+          <origin xyz="0 0 ${-(height3 - axel_offset*2)}" rpy="0 0 0" />
+          <parent link="${prefix}link3"/>
           <child link="${prefix}tool_link" />
         </joint>
