Commit message: got data for part 3, tuned PI gains

File: rrbot_simulation_files/rrbot_description/urdf/rrbot_description.urdf.xacro (robot description, xacro)
@@ -113,5 +113,5 @@
         <axis xyz="0 0 -1"/>
         <dynamics damping="0.7"/>
-        <limit effort="300" velocity="0.1" lower="0" upper="0.50"/>
+        <limit effort="300" velocity="0.1" lower="0" upper="0"/>
       </joint>
       <!-- Link 3 -->
